File: nomech_mini.sch (KiCad schematic (older format))
At the start: 15 parts

Commit message: working mainly on LEDs
Connections:
- net labels added: AN_1, AN_2, AN_3, AN_4, LED_COLUMN_1, LED_COLUMN_2, LED_COLUMN_3, LED_COLUMN_4, LED_ROW_1, LED_ROW_2, LED_ROW_3, LED_ROW_4
- wire segments 77 -> 101
Other:
- moved on the sheet: C?, L?
Changed lines of the file:
@@
-EESchema Schematic File Version 2  date Tue 09 Apr 2013 21:23:41 BST
+EESchema Schematic File Version 2  date Tue 09 Apr 2013 22:30:20 BST
 LIBS:power
 LIBS:device
@@
 L INDUCTOR L?
 U 1 1 5156DFE5
-P 6700 5250
-F 0 "L?" V 6650 5250 40  0000 C CNN
-F 1 "FERRITE_BEAD" V 6800 5250 40  0000 C CNN
-F 2 "" H 6700 5250 60  0001 C CNN
-F 3 "" H 6700 5250 60  0001 C CNN
-	1    6700 5250
+P 6900 5250
+F 0 "L?" V 6850 5250 40  0000 C CNN
+F 1 "FERRITE_BEAD" V 7000 5250 40  0000 C CNN
+F 2 "" H 6900 5250 60  0001 C CNN
+F 3 "" H 6900 5250 60  0001 C CNN
+	1    6900 5250
 	1    0    0    -1
 $EndComp
@@
 L C C?
 U 1 1 5156DFF1
-P 6700 5850
-F 0 "C?" H 6750 5950 50  0000 L CNN
-F 1 "100nF" H 6750 5750 50  0000 L CNN
-F 2 "" H 6700 5850 60  0001 C CNN
-F 3 "" H 6700 5850 60  0001 C CNN
-	1    6700 5850
+P 6900 5850
+F 0 "C?" H 6950 5950 50  0000 L CNN
+F 1 "100nF" H 6950 5750 50  0000 L CNN
+F 2 "" H 6900 5850 60  0001 C CNN
+F 3 "" H 6900 5850 60  0001 C CNN
+	1    6900 5850
 	1    0    0    -1
 $EndComp
@@
 Connection ~ 5200 7000
 Wire Wire Line
-	5200 6750 5200 7200
+	5200 6850 5200 7200
 Wire Wire Line
 	5200 7000 5150 7000
 Wire Wire Line
-	4550 6750 4550 7200
+	4550 6850 4550 7200
 Connection ~ 4550 7000
 Wire Wire Line
@@
 	5200 7800 5200 7600
 Wire Wire Line
-	4550 6750 4800 6750
-Wire Wire Line
-	4800 6750 4800 6350
-Wire Wire Line
-	5200 6750 4900 6750
-Wire Wire Line
-	4900 6750 4900 6350
+	4550 6850 4800 6850
+Wire Wire Line
+	4800 6850 4800 6350
+Wire Wire Line
+	5200 6850 4900 6850
+Wire Wire Line
+	4900 6850 4900 6350
 Wire Wire Line
 	4700 6350 4700 6500
@@
 Connection ~ 4600 3500
 Wire Wire Line
-	6700 5550 6700 5650
-Wire Wire Line
-	6050 5600 6700 5600
-Connection ~ 6700 5600
+	6900 5550 6900 5650
+Wire Wire Line
+	6050 5600 6900 5600
+Connection ~ 6900 5600
 $Comp
 L GND #PWR?
@@
 	6200 5700 6200 6100
 Wire Wire Line
-	6200 6100 6700 6100
-Wire Wire Line
-	6700 6050 6700 6150
+	6200 6100 6900 6100
 Connection ~ 6700 6100
 $Comp
 L +5V #PWR?
 U 1 1 5156E2D4
-P 6700 4850
-F 0 "#PWR?" H 6700 4940 20  0001 C CNN
-F 1 "+5V" H 6700 4940 30  0000 C CNN
-F 2 "" H 6700 4850 60  0000 C CNN
-F 3 "" H 6700 4850 60  0000 C CNN
-	1    6700 4850
-	1    0    0    -1
-$EndComp
-Wire Wire Line
-	6700 4850 6700 4950
+P 6900 4850
+F 0 "#PWR?" H 6900 4940 20  0001 C CNN
+F 1 "+5V" H 6900 4940 30  0000 C CNN
+F 2 "" H 6900 4850 60  0000 C CNN
+F 3 "" H 6900 4850 60  0000 C CNN
+	1    6900 4850
+	1    0    0    -1
+$EndComp
+Wire Wire Line
+	6900 4850 6900 4950
 $Sheet
 S 8400 4200 650  600
@@
 F1 "LEDS.sch" 50
 $EndSheet
+Text Label 3750 5600 2    60   ~ 0
+ISP_MOSI
+Text Label 3750 5700 2    60   ~ 0
+ISP_MISO
+Text Label 3750 5500 2    60   ~ 0
+ISP_SCK
+Text GLabel 6500 6800 2    60   Input ~ 0
+LED_COLUMN_1
+Text GLabel 6500 6650 2    60   Input ~ 0
+LED_COLUMN_2
+Text GLabel 6500 6500 2    60   Input ~ 0
+LED_COLUMN_3
+Text GLabel 6500 6350 2    60   Input ~ 0
+LED_COLUMN_4
+Text GLabel 6100 5200 2    60   Input ~ 0
+LED_ROW_1
+Text GLabel 6100 5000 2    60   Input ~ 0
+LED_ROW_3
+Text GLabel 4000 6250 0    60   Input ~ 0
+LED_ROW_4
+Wire Wire Line
+	5000 6350 5000 6800
+Wire Wire Line
+	5100 6350 5100 6650
+Wire Wire Line
+	5000 6800 6500 6800
+Wire Wire Line
+	5100 6650 6500 6650
+Wire Wire Line
+	5200 6350 5200 6500
+Wire Wire Line
+	5200 6500 6500 6500
+Wire Wire Line
+	5300 6350 5300 6450
+Wire Wire Line
+	5300 6450 6400 6450
+Wire Wire Line
+	6400 6450 6400 6350
+Wire Wire Line
+	6400 6350 6500 6350
+Wire Wire Line
+	6100 5200 6050 5200
+Wire Wire Line
+	6700 6100 6700 6150
+Wire Wire Line
+	6900 6100 6900 6050
+Text GLabel 6100 5100 2    60   Input ~ 0
+LED_ROW_2
+Wire Wire Line
+	6100 5100 6050 5100
+Wire Wire Line
+	6100 5000 6050 5000
+Wire Wire Line
+	4000 6250 4200 6250
+Wire Wire Line
+	4200 6250 4200 6350
+Wire Wire Line
+	4200 6350 4400 6350
+Text GLabel 4900 4050 1    60   Input ~ 0
+AN_1
+Wire Wire Line
+	4900 4050 4900 4100
+Text GLabel 5000 4050 1    60   Input ~ 0
+AN_2
+Text GLabel 5100 4050 1    60   Input ~ 0
+AN_3
+Text GLabel 5200 4050 1    60   Input ~ 0
+AN_4
+Wire Wire Line
+	5000 4050 5000 4100
+Wire Wire Line
+	5100 4050 5100 4100
+Wire Wire Line
+	5200 4050 5200 4100
+$Comp
+L GND #PWR?
+U 1 1 516489BE
+P 3600 4700
+F 0 "#PWR?" H 3600 4700 30  0001 C CNN
+F 1 "GND" H 3600 4630 30  0001 C CNN
+F 2 "" H 3600 4700 60  0000 C CNN
+F 3 "" H 3600 4700 60  0000 C CNN
+	1    3600 4700
+	1    0    0    -1
+$EndComp
+Wire Wire Line
+	3750 4700 3750 4600
+Wire Wire Line
+	3750 4600 3600 4600
+Wire Wire Line
+	3600 4600 3600 4700
 $EndSCHEMATC

Commit message: starting layout
Parts:
- added C1, C2, C3, C5: 100nF, SM0603, symbol C
- added C11, C13, C6, C8: 10nF, SM0603, symbol C
- added C15, C16, C17, C18: 4.7nF, symbol C
- added D1: LED, symbol LED
- added E1, E10, E11, E12, E13, E14, E15, E16, E2, E3, E4, E5, E6, E7, E8, E9: CAP-ELECTRODE, symbol CAP-ELECTRODE
- added P2, P3, P4, P5, P6: CONN_1, symbol CONN_1
- added R10, R11, R12, R9: 1M, symbol R
- added R13, R14, R15, R16, R5, R6, R7, R8: 1k, symbol R
- added R4: 120R, symbol R
- gave numbers to parts that had none: 15
Connections:
- net labels added: AN_5, AN_6, AN_7, AN_8, SLOPE, X1, X2, X3, X4, Y1, Y2, Y3, Y4
- wire segments 101 -> 185
- no-connect marks 0 -> 1
Other:
- moved on the sheet: C10, C7, L1

Commit message: placing LEDS, working out laser cutting
Parts:
- C1, C11, C13, C2, C3, C5, C6, C8: footprint SM0603 -> SM0805
- C10, C12, C14, C15, C16, C17, C18, C4, C7, C9, L1, L2, R1, R10, R11, R12, R13, R14, R15, R16, R2, R3, R4, R5, R6, R7, R8, R9: footprint (none) -> SM0805
- CON1: footprint (none) -> MICRO-B_USB
- CON2: footprint AVR-ISP-6 -> pin_array_3x2
- D33: renamed from D1; footprint (none) -> KPJA-2107SURCK
- E1, E10, E11, E12, E13, E14, E15, E16, E2, E3, E4, E5, E6, E7, E8, E9: footprint (none) -> cap-electrode_10mm_2layer
- P2, P3, P4, P5, P6: footprint (none) -> PIN_ARRAY_1
- U1: footprint ~ -> TQFP44
- X1: footprint (none) -> adafruit-NX5032

Commit message: placed?
Parts:
- removed C3, C5: 100nF, SM0805, symbol C
- removed C6, C8: 10nF, SM0805, symbol C
Connections:
- wire segments 185 -> 177
Other:
- moved on the sheet: C1, C11, C13, C2
Changed lines of the file:
@@
-EESchema Schematic File Version 2  date Thu 11 Apr 2013 21:49:24 BST
+EESchema Schematic File Version 2  date Fri 12 Apr 2013 22:25:08 BST
 LIBS:power
 LIBS:device
@@
 LIBS:cap-electrode
 LIBS:nomech_mini-cache
-EELAYER 27 0
+EELAYER 24 0
 EELAYER END
 $Descr A3 16535 11693
@@
 Sheet 1 2
 Title ""
-Date "11 apr 2013"
+Date "12 apr 2013"
 Rev ""
 Comp ""
@@
 L C C13
 U 1 1 51675C86
-P 5500 9650
-F 0 "C13" H 5540 9674 70  0000 L BNN
-F 1 "10nF" H 5539 9485 70  0000 L BNN
-F 2 "SM0805" H 5539 9585 70  0001 C CNN
-F 3 "" H 5500 9650 60  0001 C CNN
-	1    5500 9650
+P 4550 9650
+F 0 "C13" H 4590 9674 70  0000 L BNN
+F 1 "10nF" H 4589 9485 70  0000 L BNN
+F 2 "SM0805" H 4589 9585 70  0001 C CNN
+F 3 "" H 4550 9650 60  0001 C CNN
+	1    4550 9650
 	1    0    0    -1
 $EndComp
@@
 L C C11
 U 1 1 51675C8C
-P 5000 9650
-F 0 "C11" H 5040 9674 70  0000 L BNN
-F 1 "10nF" H 5039 9485 70  0000 L BNN
-F 2 "SM0805" H 5039 9585 70  0001 C CNN
-F 3 "" H 5000 9650 60  0001 C CNN
-	1    5000 9650
-	1    0    0    -1
-$EndComp
-$Comp
-L C C8
-U 1 1 51675C92
-P 4500 9650
-F 0 "C8" H 4540 9674 70  0000 L BNN
-F 1 "10nF" H 4539 9485 70  0000 L BNN
-F 2 "SM0805" H 4539 9585 70  0001 C CNN
-F 3 "" H 4500 9650 60  0001 C CNN
-	1    4500 9650
+P 4050 9650
+F 0 "C11" H 4090 9674 70  0000 L BNN
+F 1 "10nF" H 4089 9485 70  0000 L BNN
+F 2 "SM0805" H 4089 9585 70  0001 C CNN
+F 3 "" H 4050 9650 60  0001 C CNN
+	1    4050 9650
 	1    0    0    -1
 $EndComp
@@
 L C C1
 U 1 1 51675C98
-P 1900 9650
-F 0 "C1" H 1940 9674 70  0000 L BNN
-F 1 "100nF" H 1939 9485 70  0000 L BNN
-F 2 "SM0805" H 1939 9585 70  0001 C CNN
-F 3 "" H 1900 9650 60  0001 C CNN
-	1    1900 9650
+P 2950 9650
+F 0 "C1" H 2990 9674 70  0000 L BNN
+F 1 "100nF" H 2989 9485 70  0000 L BNN
+F 2 "SM0805" H 2989 9585 70  0001 C CNN
+F 3 "" H 2950 9650 60  0001 C CNN
+	1    2950 9650
 	1    0    0    -1
 $EndComp
@@
 L C C2
 U 1 1 51675C9E
-P 2400 9650
-F 0 "C2" H 2440 9674 70  0000 L BNN
-F 1 "100nF" H 2439 9485 70  0000 L BNN
-F 2 "SM0805" H 2439 9585 70  0001 C CNN
-F 3 "" H 2400 9650 60  0001 C CNN
-	1    2400 9650
-	1    0    0    -1
-$EndComp
-$Comp
-L C C3
-U 1 1 51675CA4
-P 2900 9650
-F 0 "C3" H 2940 9674 70  0000 L BNN
-F 1 "100nF" H 2939 9485 70  0000 L BNN
-F 2 "SM0805" H 2939 9585 70  0001 C CNN
-F 3 "" H 2900 9650 60  0001 C CNN
-	1    2900 9650
+P 3450 9650
+F 0 "C2" H 3490 9674 70  0000 L BNN
+F 1 "100nF" H 3489 9485 70  0000 L BNN
+F 2 "SM0805" H 3489 9585 70  0001 C CNN
+F 3 "" H 3450 9650 60  0001 C CNN
+	1    3450 9650
 	1    0    0    -1
 $EndComp
@@
 F 3 "" H 3700 9250 60  0001 C CNN
 	1    3700 9250
-	1    0    0    -1
-$EndComp
-$Comp
-L C C6
-U 1 1 51675CB6
-P 3950 9650
-F 0 "C6" H 3990 9674 70  0000 L BNN
-F 1 "10nF" H 3989 9485 70  0000 L BNN
-F 2 "SM0805" H 3989 9585 70  0001 C CNN
-F 3 "" H 3950 9650 60  0001 C CNN
-	1    3950 9650
-	1    0    0    -1
-$EndComp
-$Comp
-L C C5
-U 1 1 51675CBC
-P 3450 9650
-F 0 "C5" H 3490 9674 70  0000 L BNN
-F 1 "100nF" H 3489 9485 70  0000 L BNN
-F 2 "SM0805" H 3489 9585 70  0001 C CNN
-F 3 "" H 3450 9650 60  0001 C CNN
-	1    3450 9650
 	1    0    0    -1
 $EndComp
@@
 Wire Wire Line
 	3700 9900 3700 10100
-Connection ~ 4500 9900
 Connection ~ 3450 9900
-Connection ~ 2400 9900
-Connection ~ 2400 9400
-Wire Wire Line
-	1900 9400 5500 9400
 Connection ~ 3450 9400
-Connection ~ 5000 9400
-Connection ~ 3950 9400
+Wire Wire Line
+	2950 9400 4550 9400
+Connection ~ 4050 9400
 Wire Wire Line
 	3700 9400 3700 9250
-Connection ~ 4500 9400
 Connection ~ 3700 9400
-Connection ~ 2900 9400
-Connection ~ 2900 9900
-Connection ~ 3950 9900
-Wire Wire Line
-	1900 9900 5500 9900
-Connection ~ 5000 9900
-Wire Wire Line
-	1900 9400 1900 9450
-Wire Wire Line
-	1900 9900 1900 9850
-Wire Wire Line
-	2400 9400 2400 9450
-Wire Wire Line
-	2400 9900 2400 9850
-Wire Wire Line
-	2900 9900 2900 9850
-Wire Wire Line
-	2900 9400 2900 9450
+Wire Wire Line
+	2950 9900 4550 9900
+Connection ~ 4050 9900
+Wire Wire Line
+	2950 9400 2950 9450
+Wire Wire Line
+	2950 9900 2950 9850
 Wire Wire Line
 	3450 9400 3450 9450
@@
 Connection ~ 10700 7950
 Wire Wire Line
-	3950 9450 3950 9400
-Wire Wire Line
-	3950 9850 3950 9900
-Wire Wire Line
-	4500 9450 4500 9400
-Wire Wire Line
-	4500 9850 4500 9900
-Wire Wire Line
-	5000 9450 5000 9400
-Wire Wire Line
-	5000 9850 5000 9900
-Wire Wire Line
-	5500 9400 5500 9450
-Wire Wire Line
-	5500 9900 5500 9850
+	4050 9450 4050 9400
+Wire Wire Line
+	4050 9850 4050 9900
+Wire Wire Line
+	4550 9400 4550 9450
+Wire Wire Line
+	4550 9900 4550 9850
 Wire Wire Line
 	5400 3950 5400 4100

Commit message: laying out 4 types of LED+electrode combos
Parts:
- D1: renamed from D33; footprint KPJA-2107SURCK -> SM0402
- E1, E10, E11, E12, E13, E14, E15, E16, E2, E3, E4, E5, E6, E7, E8, E9: footprint cap-electrode_10mm_2layer -> cap-electrode_16mm
- renumbered C7 to C1, C18 to C10, C1 to C11, C2 to C12, C11 to C13, C13 to C14, C10 to C2, C15 to C3, C16 to C5, C14 to C6, C17 to C7, C9 to C8, C12 to C9, P3 to P1, P4 to P2, P5 to P3, P2 to P4, P6 to P5, R4 to R1, R14 to R10, R10 to R11, R15 to R12, R1 to R13, R11 to R14, R16 to R15, R12 to R16, R13 to R2, R5 to R3, R6 to R4, R9 to R5, R7 to R6, R2 to R7, R3 to R9
